Commit message: ergerger

File: resources/urdf/rrbot.xacro (robot description, xacro)
@@ -12,7 +12,7 @@
   <xacro:property name="axel_offset" value="0.05" /> <!-- Space btw top of beam and the each joint -->
   <!-- Import all Gazebo-customization elements, including Gazebo colors -->
-  <xacro:include filename="$(find rrbot_description)/urdf/rrbot.gazebo" />
+  <xacro:include filename="$(find ros_rrbot_lecture)/resources/urdf/rrbot.gazebo" />
   <!-- Import Rviz colors -->
-  <xacro:include filename="$(find rrbot_description)/urdf/materials.xacro" />
+  <xacro:include filename="$(find ros_rrbot_lecture)/resources/urdf/materials.xacro" />
   <!-- Used for fixing robot to Gazebo 'base_link' -->
   <link name="world"/>
@@ -124,5 +124,5 @@
       <origin xyz="0 0 0" rpy="0 0 0"/>
       <geometry>
-        <mesh filename="package://rrbot_description/meshes/hokuyo.dae"/>
+        <mesh filename="package://ros_rrbot_lecture/resources/meshes/hokuyo.dae"/>
       </geometry>
     </visual>

Commit message: final details

File: resources/urdf/rrbot.xacro (robot description, xacro)
@@ -11,4 +11,5 @@
   <xacro:property name="camera_link" value="0.05" /> <!-- Size of square 'camera' box -->
   <xacro:property name="axel_offset" value="0.05" /> <!-- Space btw top of beam and the each joint -->
+  <xacro:property name="joint_damping" value="0.05" /> <!-- Damping coefficient of each joint -->
   <!-- Import all Gazebo-customization elements, including Gazebo colors -->
   <xacro:include filename="$(find ros_rrbot_lecture)/resources/urdf/rrbot.gazebo" />
@@ -50,5 +51,5 @@
     <origin xyz="0 ${width} ${height1 - axel_offset}" rpy="0 0 0"/>
     <axis xyz="0 1 0"/>
-    <dynamics damping="0.7"/>
+    <dynamics damping="${joint_damping}"/>
   </joint>
   <!-- Middle Link -->
@@ -81,5 +82,5 @@
     <origin xyz="0 ${width} ${height2 - axel_offset*2}" rpy="0 0 0"/>
     <axis xyz="0 1 0"/>
-    <dynamics damping="0.7"/>
+    <dynamics damping="${joint_damping}"/>
   </joint>
   <!-- Top Link -->
